File: hardware/pcb/tethos-pet.kicad_pcb (KiCad board)
At the start: 4 copper layers, 48.4 x 38.4 mm, 27 parts, among them J1 AFA07-S14FCA-00, Q1 2N7002, Q2 AO3401A, SW1 SKRTLAE010, SW2 SKRTLAE010, SW3 SKRTLAE010, SW4 SKRTLAE010, U1 ANNA-B112, Y1 32.768kHz 12.5pF 3215

Commit message: J1: dual-contact FPC, nets mirrored for the folded ribbon
ERC12864-9 outline (third-angle): LCD pin 1 is on the right seen from the front and the
tail contacts are on the back face. After the 180 deg fold behind the LCD the contacts face
away from the PCB and pin 1 lands on the right, so the bottom-contact AFA07 with pad n = pin n
would not have worked.

- J1 -> HDGC 1.0-B-14PWB (C2915494), contacts top and bottom, 2.85 mm
- pad k = LCD pin 15-k; pads at z 8.5 so the ribbon tip gets ~3 mm insertion
- LCD gap 2.8 -> 3.1 mm, shell depth 18.1 -> 18.4 mm; rerouted, DRC 0/0, fit check clean
- JLC CPL: J1 needs no correction with this footprint

Co-Authored-By: Claude Opus 5.5 <noreply@anthropic.com>
Parts:
- J1: value AFA07-S14FCA-00 -> 1.0-B-14PWB; footprint JUSHUO_AFA07-S14FCA-00_1x14-1MP_P1.0mm_Horizontal -> FPC-SMD_14P-P1.00_HDGC_1.0-B-14PWB
- moved J1 2.20 mm to (0.00, -8.50)
Connections:
- J1 pad 1: (no net) -> LCD_VG
- J1 pad 10: LCD_V0 -> LCD_A0
- J1 pad 11: LCD_XV0 -> LCD_RST
- J1 pad 12: (no net) -> LCD_CS
- J1 pad 14: LCD_VG -> (no net)
- J1 pad 3: LCD_CS -> (no net)
- J1 pad 4: LCD_RST -> LCD_XV0
- J1 pad 5: LCD_A0 -> LCD_V0
- J1 pad 6: LCD_SCL -> GND
- J1 pad 7: LCD_SDA -> VBAT
- J1 pad 8: VBAT -> LCD_SDA
- J1 pad 9: GND -> LCD_SCL
Routing:
- net LCD_VG: track 2.04 -> 17.8 mm
- net GND: track 77.4 -> 62.8 mm
- net LCD_CS: track 3.70 -> 14.4 mm
- net LCD_RST: track 6.28 -> 14.8 mm
- net LCD_XV0: track 2.04 -> 9.33 mm, vias 0 -> 2
- net BUZZ_G: track 12.7 -> 6.65 mm
- net LCD_SDA: track 8.02 -> 13.8 mm
- net LCD_V0: track 2.04 -> 7.52 mm, vias 0 -> 2
- net LCD_A0: track 5.34 -> 9.95 mm
- net BTN_C: track 33.0 -> 28.7 mm, vias 2 -> 0
- net LCD_SCL: track 16.7 -> 20.3 mm
- net XL1: track 11.5 -> 8.30 mm
- net BUZZ: track 27.4 -> 24.9 mm
- net VCELL: track 40.9 -> 42.6 mm, vias 0 -> 2
- net BTN_A: track 17.8 -> 16.2 mm, vias 2 -> 0
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